File: PCB/quackpad.kicad_sch (KiCad schematic)
At the start: 28 parts, among them SW1 SW_Push, SW10 SW_Push, SW11 SW_Push, SW12 SW_Push, SW13 SW_Push, SW2 SW_Push, SW3 SW_Push, SW4 SW_Push, SW5 SW_Push, SW6 SW_Push, SW7 SW_Push, SW8 SW_Push, SW9 SW_Push, U1 MOUDLE-SEEEDUINO-XIAO

Commit message: Add files via upload
Parts:
- removed D9: 1N4148, Diode_THT:D_DO-35_SOD27_P7.62mm_Horizontal, symbol Diode:1N4148
- removed SW2: SW_Push, symbol Switch:SW_Push
- added J1: OLED_128x32, ScottoKeebs_Components:OLED_128x32, symbol ScottoKeebs:OLED_128x32
Connections:
- net GND: now also J1.1 (GND)
- net VCC: now also U1.14 (5V), J1.2 (VCC)
- net SDA: now reaches U1.5 (PA8_A4_D4_SDA)
- net SCL: now reaches U1.6 (PA9_A5_D5_SCL)
- net row 3: no longer names the net of U1.8 (PB09_A7_D7_RX)
